Commit message: release: v0.6.1 scene loading, gripper, and grasp smoke
Ship MobileManipulatorSim scene paths, parallel-jaw gripper on mm_minimal, example 22 grasp contact CI, and wire viewer/ROS/reach to scene assets.

File: assets/robots/mm_minimal/mm_minimal.urdf (robot description, URDF)
Before this commit: robot mm_minimal, 3 links, 2 joints
Links:
- added link gripper_base_link; collision box size=0.06 0.04 0.04; visual box size=0.06 0.04 0.04
- added link left_finger_link; collision box size=0.02 0.02 0.08; visual box size=0.02 0.02 0.08
- added link right_finger_link; collision box size=0.02 0.02 0.08; visual box size=0.02 0.02 0.08
Joints:
- added joint gripper_base_joint: type fixed, parent forearm_link, child gripper_base_link, origin xyz=0.4 0 0 rpy=0 0 0
- added joint left_finger_joint: type revolute, parent gripper_base_link, child left_finger_link, origin xyz=0 0 -0.04 rpy=0 0 0, axis 0 1 0
- added joint right_finger_joint: type revolute, parent gripper_base_link, child right_finger_link, origin xyz=0 0 0.04 rpy=0 0 0, axis 0 1 0
