Commit message: fix(rne_ai): stabilize mm_minimal settle physics and re-derive fixed-base tasks
The fixed-base SCARA arm never settled: its base/upper-arm/forearm colliders
interpenetrated (injecting contact energy every tick) and its shoulder/elbow
were bare velocity motors with no restoring force, so the idle pose was a
sustained chaotic oscillation that Windows and Linux merely sampled at
different points. Mirror the proven mm_mobile fix and re-derive the tasks
that had been tuned against the chaos:

- mm_minimal.urdf: trim the chassis/upper-arm/forearm collision boxes so
  adjacent links no longer interpenetrate (visuals unchanged), and shrink the
  gripper mount collider to a token box: a full-size mount collider ejects any
  graspable object from between the fingers before they can close on it.
- sim.rs: give the fixed-base shoulder/elbow the same spring-damper position
  hold as mm_mobile/mm_lift (configure_arm_position_motors), extend the
  anti-windup lead to all velocity-integrated arms (keyed on !has_lift so
  mm_lift's direct-IK targets stay unchanged), and seat the fixed-base grasp
  weld 2 cm upward: the SCARA cannot lift, and a weld at exactly the object's
  resting height pins its support contact into the constraint system, which
  resists a horizontal carry far harder than sliding friction.
- Clutter scene/tasks: the old cube layout (x 1.05-1.22) was only pickable
  because the unstable arm stretched its impulse joints past the 0.9 m
  kinematic reach limit; re-home the cubes inside the analytic workspace with
  clean approach/carry lanes, add an elbow-down IK branch so the approach
  folds the fingertips onto the cube instead of bulldozing it with the
  forearm, and drive approach/carry with IK position tracking instead of the
  old bang-bang law (a relay oscillator against the new position-held servo).
- Place targets: re-derive to where the stable scripted rollouts actually set
  the cube down (the lift task's existing convention); the old transport
  place target (1.23, -0.53) was beyond kinematic reach and only ever hit by
  chaos-flung cubes.
- mm_minimal_transport scene: support the grasp cube on a small fixed table
  so the scripted grasp no longer depends on catching a free-falling cube
  within its first few ticks.

mm_mobile and mm_lift dynamics are untouched (hero digest unaffected).

Co-Authored-By: Claude Fable 5 <noreply@anthropic.com>
Claude-Session: https://claude.ai/code/session_01BeQ8A66oDCEMhHgu8fDBLQ

File: assets/robots/mm_minimal/mm_minimal.urdf (robot description, URDF)
Before this commit: robot mm_minimal, 6 links, 5 joints
Links:
- link base_link: geometry collision box size=0.4 0.5 0.4; visual box size=0.4 0.6 0.4
- link forearm_link: geometry collision box size=0.34 0.06 0.06; visual box size=0.4 0.06 0.06
- link gripper_base_link: geometry collision box size=0.005 0.005 0.005; visual box size=0.06 0.04 0.04
- link upper_arm_link: geometry collision box size=0.46 0.08 0.08; visual box size=0.5 0.08 0.08
