Commit message: feat: column base lets the lift lower the gripper to the ground
Manipulator-redesign phase 1. The mm_lift robot is rebuilt on a tall fixed
column with the arm hanging from a sliding carriage, so the lift can lower
the gripper from its rest height (~0.81 m) down to near the ground (~0.26 m)
and raise it to carry. The previous box base sat under the carriage, so the
lift could only travel up. The arm also settles much straighter on the new
geometry.

Widen the lift travel limits (-0.5..0.5 m) and add a test
(lift_lowers_gripper_toward_ground). All existing mm_lift tests, the example
30 smoke, asset validation, and the determinism test pass.

File: assets/robots/mm_lift/mm_lift.urdf (robot description, URDF)
Before this commit: robot mm_lift, 7 links, 6 joints
Links:
- link base_link: geometry collision box size=0.16 1.5 0.16; visual box size=0.16 1.5 0.16
- link torso_link: geometry collision box size=0.14 0.14 0.14; visual box size=0.14 0.14 0.14
Joints:
- joint lift_joint: origin xyz=0 0.38 0 rpy=0 0 0 -> xyz=0.15 0.15 0 rpy=0 0 0

Commit message: feat: make the lift robot arm controllable (redesign P2)
The heavy lift-robot arm could not be positioned: a velocity motor (gain
1.0) was too weak to move or hold it, so a shoulder command barely turned
the arm. Two fixes:

- The upper arm's collision box overlapped the carriage (torso_link),
  jamming the shoulder. Offset the shoulder joint out along the arm so it
  clears the carriage; the arm now also settles perfectly straight.
- Drive the arm's shoulder/elbow with position (spring-damper) motors and
  a raised torque cap so the arm moves to a commanded angle and holds it.

Add a per-motor force override (JointMotor.max_force, default 0.0 = use the
per-joint-type cap) so the arm joints can apply more torque than the 50 N·m
revolute default without affecting other robots. New test
lift_arm_tracks_and_holds_commanded_pose; all existing tests/smokes pass.

File: assets/robots/mm_lift/mm_lift.urdf (robot description, URDF)
Before this commit: robot mm_lift, 7 links, 6 joints
Joints:
- joint shoulder_joint: origin xyz=0 0 0 rpy=0 0 0 -> xyz=0.16 0 0 rpy=0 0 0

Commit message: feat: top-down claw picks a ground cube and lifts it (redesign P3)
Redesign the mm_lift gripper as a top-down claw: the gripper body sits
above the object and two long fingers hang down to straddle it, so the
arm can lower the claw over a cube on the ground, grasp it (contact-
triggered weld), and the lift raises it off the ground. The previous
side-grip could not pick a ground object — its body occupied the grasp
volume and collided with the cube.

Add the mm_lift_pick scene (cube on the ground under the gripper),
mm_lift_pick_scene_path(), and a test that lowers, grasps, and lifts the
cube ~0.9 m off the ground. Wired into asset validation; full ci passes.

File: assets/robots/mm_lift/mm_lift.urdf (robot description, URDF)
Before this commit: robot mm_lift, 7 links, 6 joints
Links:
- link gripper_base_link: geometry collision box size=0.06 0.04 0.12; visual box size=0.06 0.04 0.12
- link left_finger_link: geometry collision box size=0.02 0.20 0.02; visual box size=0.02 0.20 0.02
- link right_finger_link: geometry collision box size=0.02 0.20 0.02; visual box size=0.02 0.20 0.02
Joints:
- joint left_finger_joint: axis 0 1 0 -> 1 0 0; origin xyz=0 0 -0.04 rpy=0 0 0 -> xyz=0 -0.02 -0.045 rpy=0 0 0
- joint right_finger_joint: axis 0 1 0 -> 1 0 0; origin xyz=0 0 0.04 rpy=0 0 0 -> xyz=0 -0.02 0.045 rpy=0 0 0
