Commit message: feat: pick&place weld grasp, RL bindings, ROS gripper/TF, mm_mobile wheel fix
Physics:
- Add prismatic and fixed (weld) joints to rne_physics + Rapier backend
- Make backend ECS iteration deterministic (body/joint sync + transform
  write-back sorted by entity), fixing the flaky shoulder-motor test

Manipulation (Phase C):
- Contact-triggered weld grasp in MobileManipulatorSim (is_grasping/grasped_object):
  closing the gripper onto a body welds it to the end-effector, opening releases it
- MobileManipulatorTask::Place + MobileManipulatorEpisodeConfig::place()
- Example 26 pick-and-place smoke (grasp -> carry -> release -> settle)
- Recalibrate example 21 reach target to the now-deterministic reachable pose

RL / Python:
- rne_py MobileManipulator bindings (sim + episode, place/transport/inspect)
- Example 27 gymnasium-style MobileManipulatorPlaceEnv (degrades without gymnasium/numpy)

ROS 2:
- /gripper_command (std_msgs/Float64) and ee_link TF in mobile_manipulator mode
- Fix rne_ros2_node build: sensor_msgs/Image.is_bigendian bool -> u8
- Smoke checks peak |base_x| (mm_mobile path curves) + gripper/ee_link

Assets:
- Fix mm_mobile drive wheels: were stacked vertically (only one touched ground,
  base spun in place); relocated to a proper left/right diff-drive layout so the
  base drives forward

Verified: cargo run -p xtask -- ci and cargo run -p xtask -- ci-ros2 both pass.

File: assets/robots/mm_mobile/mm_mobile.urdf (robot description, URDF)
Before this commit: robot mm_mobile, 5 links, 4 joints
Joints:
- joint left_wheel_joint: origin xyz=0 0.225 0 rpy=0 0 0 -> xyz=0 -0.15 0.225 rpy=0 0 0
- joint right_wheel_joint: origin xyz=0 -0.225 0 rpy=0 0 0 -> xyz=0 -0.15 -0.225 rpy=0 0 0

Commit message: feat: make README hero carry a task object

File: assets/robots/mm_mobile/mm_mobile.urdf (robot description, URDF)
Before this commit: robot mm_mobile, 5 links, 4 joints
Links:
- added link gripper_base_link; visual box size=0.06 0.04 0.04
- added link left_finger_link; visual box size=0.02 0.02 0.08
- added link right_finger_link; visual box size=0.02 0.02 0.08
Joints:
- added joint gripper_base_joint: type fixed, parent forearm_link, child gripper_base_link, origin xyz=0.4 0 0 rpy=0 0 0
- added joint left_finger_joint: type revolute, parent gripper_base_link, child left_finger_link, origin xyz=0 0 -0.04 rpy=0 0 0, axis 0 1 0
- added joint right_finger_joint: type revolute, parent gripper_base_link, child right_finger_link, origin xyz=0 0 0.04 rpy=0 0 0, axis 0 1 0
