Commit message: feat(rne_ai): complete mobile clutter navigate-grasp-place E2E
- add missing gripper/finger collision geometry to mm_mobile.urdf and
  trim chassis/arm collision boxes so jointed neighbors no longer
  interpenetrate (arm was frozen by contact impulses)
- lower mm_mobile_clutter table/cubes to the lift-less arm's shoulder plane
- drive the pinned mobile base kinematically from the commanded twist with
  planar +X yaw projection (deterministic heading, no Euler aliasing)
- position-hold motors + anti-windup lead on the mobile arm joints
- rewrite IkMobileClutterPickPlacePolicy as an observation-gated phase
  machine (settle, pick drive, carry drive, place swing, release) with
  grasp-offset-corrected base-frame IK place targets
- un-ignore mobile_clutter_policy_completes_place and
  mobile_clutter_transport_script_places_cube_a; add sim regression tests
  for finger articulation and arm joint tracking
- roadmap: add v0.13 goal (mobile clutter place E2E); changelog under
  Unreleased

Co-Authored-By: Claude Fable 5 <noreply@anthropic.com>
Claude-Session: https://claude.ai/code/session_01BeQ8A66oDCEMhHgu8fDBLQ

File: assets/robots/mm_mobile/mm_mobile.urdf (robot description, URDF)
Before this commit: robot mm_mobile, 8 links, 7 joints
Links:
- link base_link: geometry collision box size=0.5 0.2 0.4; visual box size=0.5 0.3 0.4
- link forearm_link: geometry collision box size=0.34 0.06 0.06; visual box size=0.4 0.06 0.06
- link gripper_base_link: geometry collision box size=0.06 0.04 0.04; visual box size=0.06 0.04 0.04
- link left_finger_link: geometry collision box size=0.02 0.02 0.08; visual box size=0.02 0.02 0.08
- link right_finger_link: geometry collision box size=0.02 0.02 0.08; visual box size=0.02 0.02 0.08
- link upper_arm_link: geometry collision box size=0.46 0.08 0.08; visual box size=0.5 0.08 0.08
