Commit message: Improve README hero URDF visuals

File: assets/robots/mm_mobile/mm_mobile.urdf (robot description, URDF)
Before this commit: robot mm_mobile, 8 links, 7 joints
Links:
- link forearm_link: geometry collision box size=0.34 0.06 0.06; visual box size=0.4 0.055 0.055
- link gripper_base_link: geometry collision box size=0.06 0.04 0.04; visual box size=0.10 0.07 0.09
- link upper_arm_link: geometry collision box size=0.46 0.08 0.08; visual box size=0.5 0.07 0.07
