Commit message: feat: prepare 0.1.0 release with mobile lift

File: crates/rne_urdf_import/tests/fixtures/prismatic_slider.urdf (robot description, URDF)
Before this commit: robot prismatic_slider, 2 links, 1 joints
Joints:
- joint slider_joint: limit (none) -> lower=0.0 upper=0.15 effort=20.0 velocity=0.5
