Commit message: feat(assets): ship authored mobile manipulator PBR visuals

File: assets/robots/mm_mobile_lift/mm_mobile_lift.urdf (robot description, URDF)
Before this commit: robot mm_mobile_lift, 10 links, 9 joints
Links:
- link base_link: geometry collision box size=0.5 0.2 0.4; visual mesh filename=meshes/base_link.lod0.glb scale=1 1 1
- link forearm_link: geometry collision box size=0.28 0.04 0.04; visual mesh filename=meshes/forearm_link.lod0.glb scale=1 1 1
- link gripper_base_link: geometry collision box size=0.02 0.02 0.01; visual mesh filename=meshes/gripper_base_link.lod0.glb scale=1 1 1
- link left_finger_link: geometry collision box size=0.12 0.07 0.02; visual mesh filename=meshes/left_finger_link.lod0.glb scale=1 1 1
- link left_wheel: geometry visual mesh filename=meshes/left_wheel.lod0.glb scale=1 1 1
- link right_finger_link: geometry collision box size=0.12 0.07 0.02; visual mesh filename=meshes/right_finger_link.lod0.glb scale=1 1 1
- link right_wheel: geometry visual mesh filename=meshes/right_wheel.lod0.glb scale=1 1 1
- link torso_link: geometry collision box size=0.08 0.08 0.08; visual mesh filename=meshes/torso_link.lod0.glb scale=1 1 1
- link upper_arm_link: geometry collision box size=0.42 0.035 0.035; visual mesh filename=meshes/upper_arm_link.lod0.glb scale=1 1 1
- link wrist_link: geometry collision box size=0.04 0.04 0.04; visual mesh filename=meshes/wrist_link.lod0.glb scale=1 1 1

Commit message: feat(readme): add wrist rgbd manipulation view

File: assets/robots/mm_mobile_lift/mm_mobile_lift.urdf (robot description, URDF)
Before this commit: robot mm_mobile_lift, 10 links, 9 joints
Links:
- added link wrist_camera_link
Joints:
- added joint wrist_camera_joint: type fixed, parent gripper_base_link, child wrist_camera_link, origin xyz=0.10 0.06 0 rpy=-1.45 -1.5707963267948966 -0.16
