Commit message: feat(urdf): proper URDF robot visuals via importer-compatible authoring
Inline material colors (named refs fall back to gray), box/cylinder primitives instead of meshes (importer mis-scales mesh visuals), and RNE-frame origins for joints. Physics unchanged (URDF). Adds robot-preview mode.

File: assets/robots/mesh_diff_drive/mesh_diff_drive_nav.urdf (robot description, URDF)
Before this commit: robot mesh_diff_drive_nav, 3 links, 2 joints
Links:
- link base_link: geometry collision box size=0.5 0.3 0.4; visual box size=0.005 0.03 0.04
- link left_wheel: geometry collision cylinder length=0.05 radius=0.1
- link right_wheel: geometry collision cylinder length=0.05 radius=0.1
