Commit message: feat(examples): the Go2 turns the door knob with a gripper, and the door latches
The Go2 squares up to the knob, closes a two-finger gripper on it, holds it
only once both fingers are measured on it (asserted every held step), turns
it with the wrist roll until the latch lets go, pushes the leaf off its
catch, and lets go; after walking through it shuts the door until the latch
catches. All seven runs with the approach's stopping point moved over 0.3 m
pass.

- unitree_go2_arm: generic 5-DOF arm with a two-finger gripper (1.46 kg),
  generated by tools/generate_go2_arm_urdf.py; swing_door gains a knob.
- UnitreeGo2ModelTrot::stand holds the Go2 on four feet while the arm works.
- rne_physics_rapier welds links that have their own revolute or prismatic
  multibody joint as a loop-closing impulse joint (such welds were ignored).
- Example 132 matches a scan at least once a second and rejects weak matches;
  the showcase GIF adds a close-up of the hand on the knob.

File: assets/robots/go2_description/go2_arm.rne.urdf (robot description, URDF)
Before this commit: robot go2_description, 47 links, 46 joints
Links:
- added link arm_finger_left, mass 0.03; collision box size=0.05 0.012 0.03; visual box size=0.05 0.012 0.03
- added link arm_finger_right, mass 0.03; collision box size=0.05 0.012 0.03; visual box size=0.05 0.012 0.03
- added link arm_hand, mass 0.15; collision box size=0.05 0.10 0.05; visual box size=0.05 0.10 0.05
- link arm_wrist: mass 0.2 -> 0.15; geometry visual cylinder length=0.06 radius=0.025
Joints:
- added joint arm_finger_left_joint: type prismatic, parent arm_hand, child arm_finger_left, origin xyz=0.05 0 0 rpy=0 0 0, axis 0 1 0, limit lower=0.0 upper=0.04 effort=40.0 velocity=0.2
- added joint arm_finger_right_joint: type prismatic, parent arm_hand, child arm_finger_right, origin xyz=0.05 0 0 rpy=0 0 0, axis 0 -1 0, limit lower=0.0 upper=0.04 effort=40.0 velocity=0.2
- added joint arm_roll_joint: type revolute, parent arm_wrist, child arm_hand, origin xyz=0.06 0 0 rpy=0 0 0, axis 1 0 0, limit lower=-2.0 upper=2.0 effort=5.0 velocity=4.0

File: assets/robots/swing_door/swing_door.urdf (robot description, URDF)
Before this commit: robot swing_door, 2 links, 1 joints
Links:
- added link door_knob, mass 0.3; collision cylinder length=0.03 radius=0.011; collision cylinder length=0.03 radius=0.011
- link door_leaf: geometry collision box size=0.03 0.96 0.90; visual box size=0.03 0.96 0.90
Joints:
- added joint door_knob_joint: type revolute, parent door_leaf, child door_knob, origin xyz=0 -0.87 0.58 rpy=0 0 0, axis 1 0 0, limit lower=-1.2 upper=1.2 effort=0 velocity=6.0
